File: stepper_drivers.kicad_sch (KiCad schematic)
At the start: 10 parts, among them U301 DRV8833PWP, U302 DRV8833PWP

Commit message: Finished Rev A1 PCB
Added all components and routed parts for Rev A1 PCB
Parts:
- D301, D302: footprint Diode_SMD:D_0603_1608Metric -> LED_SMD:LED_0603_1608Metric
Connections:
- net LED_A: no longer names the net of D301.2 (A), R301.1
- net LED_A: no longer D302.2 (A), R302.1
- new net: D302.2 (A), R302.1
Changed lines of the file:
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@@
-		)
-	)
-	(label "LED_A"
-		(at 27.94 179.07 270)
-		(fields_autoplaced yes)
-		(effects
-			(font
-				(size 0.635 0.635)
-			)
-			(justify right bottom)
 		)
 	)
@@
 			)
 			(justify left bottom)
-		)
-	)
-	(label "LED_A"
-		(at 50.8 179.07 270)
-		(fields_autoplaced yes)
-		(effects
-			(font
-				(size 0.635 0.635)
-			)
-			(justify right bottom)
 		)
 	)
@@
 			)
 		)
-		(property "Footprint" "Diode_SMD:D_0603_1608Metric"
+		(property "Footprint" "LED_SMD:LED_0603_1608Metric"
 			(at 27.94 185.42 0)
 			(effects
@@
 			)
 		)
-		(property "Footprint" "Diode_SMD:D_0603_1608Metric"
+		(property "Footprint" "LED_SMD:LED_0603_1608Metric"
 			(at 50.8 185.42 0)
 			(effects
